File: pcb/ESP32-Zamek/power_supply.kicad_sch (KiCad schematic)
At the start: 13 parts

Commit message: Add one note
Changed lines of the file:
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@@
+		)
+	)
+	(text_box "Headery dla RFID RC522"
+		(exclude_from_sim no)
+		(at 76.2 128.905 0)
+		(size 18.415 10.795)
+		(stroke
+			(width 0)
+			(type default)
+		)
+		(fill
+			(type none)
+		)
+		(effects
+			(font
+				(size 1.27 1.27)
+			)
+			(justify left top)
 		)
 	)
@@
 		(stroke
 			(width 0)
+			(type default)
+		)
+		(fill
+			(type none)
+		)
+		(effects
+			(font
+				(size 1.27 1.27)
+			)
+			(justify left top)
+		)
+	)
+	(text_box "Port śrubowy lub DC Jack"
+		(exclude_from_sim no)
+		(at 223.52 40.64 0)
+		(size 18.415 10.795)
+		(stroke
+			(width 0)
