File: pcb/onyks_iot_control_cabinet_pcb/power_supply_nfc_connector.kicad_sch (KiCad schematic)
At the start: 13 parts

Commit message: Fix the project; cleaning up the things
Parts:
- removed C?: 100n, symbol Device:C
- removed C?: 0.1u, symbol Device:C
- removed C?: 100u, symbol Device:C
- removed C?: 2.2u, symbol Device:C
- removed J?: Conn_01x08_Socket, symbol Connector:Conn_01x08_Socket
- removed J?: Jack-DC, symbol Connector:Jack-DC
- removed J?: Screw_Terminal_01x02, symbol Connector:Screw_Terminal_01x02
- removed L?: 5.6u, symbol Device:L
- removed R? (x2): 10k, symbol Device:R
- removed R?: 100k, symbol Device:R
- removed R?: 22.1k, symbol Device:R
- removed U?: LMR51430, Package_TO_SOT_SMD:SOT-23-6, symbol Regulator_Switching:LMR51430
- added C6: 2.2u, symbol Device:C
- added C7: 100n, symbol Device:C
- added C8: 0.1u, symbol Device:C
- added C9: 100u, symbol Device:C
- added J2: Conn_01x08_Socket, symbol Connector:Conn_01x08_Socket
- added J3: Screw_Terminal_01x02, symbol Connector:Screw_Terminal_01x02
- added J4: Jack-DC, symbol Connector:Jack-DC
- added L1: 5.6u, symbol Device:L
- added R5, R6: 10k, symbol Device:R
- added R7: 100k, symbol Device:R
- added R8: 22.1k, symbol Device:R
- added U2: LMR51430, Package_TO_SOT_SMD:SOT-23-6, symbol Regulator_Switching:LMR51430
Connections:
- net +3.3V: now also C9.1, J2.8 (Pin_8), L1.2, R5.1, R6.1, R7.1
- net GND: now also C6.2, C7.2, C9.2, J2.6 (Pin_6), J3.1 (Pin_1), J4.2, R8.2, U2.1 (GND)
- net NFC_EEPROM_SCL: now also J2.2 (Pin_2), R5.2
- net NFC_EEPROM_SDA: now also J2.1 (Pin_1), R6.2
- net NFC_IRQ: now also J2.5 (Pin_5)
- net NFC_MISO: now also J2.4 (Pin_4)
- net NFC_MOSI: now also J2.3 (Pin_3)
- net NFC_RST: now also J2.7 (Pin_7)
- net V_IN: now also C6.1, C7.1, J3.2 (Pin_2), J4.1, U2.3 (VIN), U2.5 (EN)
- new net: R7.2, R8.1, U2.4 (FB)
- new net: C8.2, L1.1, U2.2 (SW)
- new net: C8.1, U2.6 (CB)
Other:
- company: (none) -> ,,Onyks'' Students Scientific Association
- title: (none) -> Onyks Iot Control Cabinet

Commit message: Assignment some footprints to symbols
Parts:
- J2: footprint (none) -> Connector_PinHeader_2.54mm:PinHeader_1x08_P2.54mm_Vertical
- J3: footprint (none) -> TerminalBlock:TerminalBlock_Xinya_XY308-2.54-2P_1x02_P2.54mm_Horizontal
- J4: footprint (none) -> Connector_BarrelJack:BarrelJack_CUI_PJ-036AH-SMT_Horizontal
- R5, R6, R7, R8: footprint (none) -> Resistor_SMD:R_0805_2012Metric_Pad1.20x1.40mm_HandSolder
Changed lines of the file:
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@@
 			)
 		)
-		(property "Footprint" ""
+		(property "Footprint" "Connector_BarrelJack:BarrelJack_CUI_PJ-036AH-SMT_Horizontal"
 			(at 212.09 64.516 0)
 			(effects
@@
 			)
 		)
-		(property "Footprint" ""
+		(property "Footprint" "Resistor_SMD:R_0805_2012Metric_Pad1.20x1.40mm_HandSolder"
 			(at 141.732 71.12 90)
 			(effects
@@
 			)
 		)
-		(property "Footprint" ""
+		(property "Footprint" "Resistor_SMD:R_0805_2012Metric_Pad1.20x1.40mm_HandSolder"
 			(at 57.912 144.78 90)
 			(effects
@@
 			)
 		)
-		(property "Footprint" ""
+		(property "Footprint" "Resistor_SMD:R_0805_2012Metric_Pad1.20x1.40mm_HandSolder"
 			(at 141.732 59.69 90)
 			(effects
@@
 			)
 		)
-		(property "Footprint" ""
+		(property "Footprint" "TerminalBlock:TerminalBlock_Xinya_XY308-2.54-2P_1x02_P2.54mm_Horizontal"
 			(at 210.82 45.72 0)
 			(effects
@@
 			)
 		)
-		(property "Footprint" ""
+		(property "Footprint" "Resistor_SMD:R_0805_2012Metric_Pad1.20x1.40mm_HandSolder"
 			(at 70.612 144.78 90)
 			(effects
@@
 			)
 		)
-		(property "Footprint" ""
+		(property "Footprint" "Connector_PinHeader_2.54mm:PinHeader_1x08_P2.54mm_Vertical"
 			(at 91.44 165.1 0)
 			(effects

Commit message: PCB - Finished, needs additional confirmation
Parts:
- removed J2: Conn_01x08_Socket, Connector_PinHeader_2.54mm:PinHeader_1x08_P2.54mm_Vertical, symbol Connector:Conn_01x08_Socket
- removed R5, R6: 10k, Resistor_SMD:R_0805_2012Metric_Pad1.20x1.40mm_HandSolder, symbol Device:R
- added J2: Conn_01x06_Socket, Connector_PinHeader_2.54mm:PinHeader_1x06_P2.54mm_Vertical, symbol Connector:Conn_01x06_Socket
- C6, C7, C8: footprint (none) -> Capacitor_SMD:C_0805_2012Metric
- C9: footprint (none) -> Capacitor_SMD:C_1210_3225Metric
- L1: footprint (none) -> ourFootprints:XAL6060-562MEC_COC
Connections:
- net +3.3V: now also J2.6 (Pin_6)
- net GND: now also J4.3, J2.4 (Pin_4)
- net NFC_IRQ: now also J2.3 (Pin_3)
- net NFC_MISO: now also J2.2 (Pin_2)
- net NFC_MOSI: now also J2.1 (Pin_1)
- net NFC_RST: now also J2.5 (Pin_5)

Commit message: Add pins for the jumper and choosing the power supply; also add connection for JTAG 3V3
Parts:
- added J5: Conn_01x03_Pin, Connector_PinHeader_2.54mm:PinHeader_1x03_P2.54mm_Vertical, symbol Connector:Conn_01x03_Pin
Connections:
- net V_IN: now also J5.2 (Pin_2); no longer J3.2 (Pin_2), J4.1
- new net: J4.1, J5.1 (Pin_1)
- new net: J3.2 (Pin_2), J5.3 (Pin_3)
Changed lines of the file:
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@@
 	(wire
 		(pts
-			(xy 215.9 43.18) (xy 222.25 43.18)
+			(xy 215.9 43.18) (xy 242.57 43.18)
 		)
 		(stroke
@@
 	(wire
 		(pts
+			(xy 242.57 60.96) (xy 242.57 54.61)
+		)
+		(stroke
+			(width 0)
+			(type default)
+		)
+	)
+	(wire
+		(pts
 			(xy 73.66 52.07) (xy 66.04 52.07)
 		)
@@
 	(wire
 		(pts
-			(xy 218.44 60.96) (xy 224.79 60.96)
+			(xy 218.44 60.96) (xy 242.57 60.96)
+		)
+		(stroke
+			(width 0)
+			(type default)
+		)
+	)
+	(wire
+		(pts
+			(xy 242.57 43.18) (xy 242.57 49.53)
 		)
 		(stroke
@@
 		(pts
 			(xy 173.99 54.61) (xy 160.02 54.61)
+		)
+		(stroke
+			(width 0)
+			(type default)
+		)
+	)
+	(wire
+		(pts
+			(xy 234.95 52.07) (xy 242.57 52.07)
 		)
 		(stroke
@@
 	(rectangle
 		(start 193.675 22.225)
-		(end 257.81 74.93)
+		(end 270.51 74.93)
 		(stroke
 			(width 0.635)
@@
 	(text_box "Terminal block/Screw port or DC Jack"
 		(exclude_from_sim no)
-		(at 234.95 46.99 0)
+		(at 246.38 34.29 0)
 		(size 18.415 10.795)
 		(stroke
@@
 	)
 	(symbol
+		(lib_id "power:+1V0")
+		(at 234.95 52.07 90)
+		(unit 1)
+		(exclude_from_sim no)
+		(in_bom yes)
+		(on_board yes)
+		(dnp no)
+		(fields_autoplaced yes)
+		(property "Reference" "#PWR024"
+			(at 238.76 52.07 0)
+			(effects
+				(font
+					(size 1.27 1.27)
+				)
+				(hide yes)
+			)
+		)
+		(property "Value" "V_IN"
+			(at 231.14 52.0699 90)
+			(effects
+				(font
+					(size 1.27 1.27)
+				)
+				(justify left)
+			)
+		)
+		(property "Footprint" ""
+			(at 234.95 52.07 0)
+			(effects
+				(font
+					(size 1.27 1.27)
+				)
+				(hide yes)
+			)
+		)
+		(property "Datasheet" ""
+			(at 234.95 52.07 0)
+			(effects
+				(font
+					(size 1.27 1.27)
+				)
+				(hide yes)
+			)
+		)
+		(property "Description" "Power symbol creates a global label with name \"+1V0\""
+			(at 234.95 52.07 0)
+			(effects
+				(font
+					(size 1.27 1.27)
+				)
+				(hide yes)
+			)
+		)
+		(pin "1"
+		)
+		(instances
+			(project "onyks_iot_control_cabinet_pcb"
+				(path "/789878cb-67d5-4bc7-a42d-b3bc72d661d0/4d976a63-6b51-465b-8a87-51604fe7b516"
+					(reference "#PWR024")
+					(unit 1)
+				)
+			)
+		)
+	)
+	(symbol
 		(lib_id "Device:L")
 		(at 127 54.61 90)
@@
 	)
 	(symbol
-		(lib_id "power:+1V0")
-		(at 224.79 60.96 270)
-		(unit 1)
-		(exclude_from_sim no)
-		(in_bom yes)
-		(on_board yes)
-		(dnp no)
-		(fields_autoplaced yes)
-		(property "Reference" "#PWR026"
-			(at 220.98 60.96 0)
-			(effects
-				(font
-					(size 1.27 1.27)
-				)
-				(hide yes)
-			)
-		)
-		(property "Value" "V_IN"
-			(at 228.6 60.9599 90)
-			(effects
-				(font
-					(size 1.27 1.27)
-				)
-				(justify left)
-			)
-		)
-		(property "Footprint" ""
-			(at 224.79 60.96 0)
-			(effects
-				(font
-					(size 1.27 1.27)
-				)
-				(hide yes)
-			)
-		)
-		(property "Datasheet" ""
-			(at 224.79 60.96 0)
-			(effects
-				(font
-					(size 1.27 1.27)
-				)
-				(hide yes)
-			)
-		)
-		(property "Description" "Power symbol creates a global label with name \"+1V0\""
-			(at 224.79 60.96 0)
-			(effects
-				(font
-					(size 1.27 1.27)
-				)
-				(hide yes)
-			)
-		)
-		(pin "1"
-		)
-		(instances
-			(project "onyks_iot_control_cabinet_pcb"
-				(path "/789878cb-67d5-4bc7-a42d-b3bc72d661d0/4d976a63-6b51-465b-8a87-51604fe7b516"
-					(reference "#PWR026")
-					(unit 1)
-				)
-			)
-		)
-	)
-	(symbol
 		(lib_id "power:GND")
 		(at 160.02 80.01 0)
@@
 	)
 	(symbol
-		(lib_id "power:+1V0")
-		(at 222.25 43.18 270)
-		(unit 1)
-		(exclude_from_sim no)
-		(in_bom yes)
-		(on_board yes)
-		(dnp no)
-		(fields_autoplaced yes)
-		(property "Reference" "#PWR024"
-			(at 218.44 43.18 0)
-			(effects
-				(font
-					(size 1.27 1.27)
-				)
-				(hide yes)
-			)
-		)
-		(property "Value" "V_IN"
-			(at 226.06 43.1799 90)
-			(effects
-				(font
-					(size 1.27 1.27)
-				)
-				(justify left)
-			)
-		)
-		(property "Footprint" ""
-			(at 222.25 43.18 0)
-			(effects
-				(font
-					(size 1.27 1.27)
-				)
-				(hide yes)
-			)
-		)
-		(property "Datasheet" ""
-			(at 222.25 43.18 0)
-			(effects
-				(font
-					(size 1.27 1.27)
-				)
-				(hide yes)
-			)
-		)
-		(property "Description" "Power symbol creates a global label with name \"+1V0\""
-			(at 222.25 43.18 0)
-			(effects
-				(font
-					(size 1.27 1.27)
-				)
-				(hide yes)
-			)
-		)
-		(pin "1"
-		)
-		(instances
-			(project "onyks_iot_control_cabinet_pcb"
-				(path "/789878cb-67d5-4bc7-a42d-b3bc72d661d0/4d976a63-6b51-465b-8a87-51604fe7b516"
-					(reference "#PWR024")
-					(unit 1)
-				)
-			)
-		)
-	)
-	(symbol
 		(lib_id "Device:R")
 		(at 143.51 59.69 0)
@@
 					(unit 1)
 				)
+			)
+		)
+	)
+	(symbol
+		(lib_id "Connector:Conn_01x03_Pin")
+		(at 247.65 52.07 180)
+		(unit 1)
+		(exclude_from_sim no)
+		(in_bom yes)
+		(on_board yes)
+		(dnp no)
+		(fields_autoplaced yes)
+		(property "Reference" "J5"
+			(at 248.92 50.7999 0)
+			(effects
+				(font
+					(size 1.27 1.27)
+				)
+				(justify right)
+			)
+		)
+		(property "Value" "Conn_01x03_Pin"
+			(at 248.92 53.3399 0)
+			(effects
+				(font
+					(size 1.27 1.27)
+				)
+				(justify right)
+			)
+		)
+		(property "Footprint" "Connector_PinHeader_2.54mm:PinHeader_1x03_P2.54mm_Vertical"
+			(at 247.65 52.07 0)
+			(effects
+				(font
+					(size 1.27 1.27)
+				)
+				(hide yes)
+			)
+		)
+		(property "Datasheet" "~"
+			(at 247.65 52.07 0)
+			(effects
+				(font
+					(size 1.27 1.27)
+				)
+				(hide yes)
+			)
+		)
+		(property "Description" "Generic connector, single row, 01x03, script generated"
+			(at 247.65 52.07 0)
+			(effects
+				(font
+					(size 1.27 1.27)
+				)
+				(hide yes)
+			)
+		)
+		(pin "3"
+		)
+		(pin "2"
+		)
+		(pin "1"
+		)
+		(instances
+			(project ""
+				(path "/789878cb-67d5-4bc7-a42d-b3bc72d661d0/4d976a63-6b51-465b-8a87-51604fe7b516"
+					(reference "J5")
+					(unit 1)
+				)
