File: pcb/onyks_iot_control_cabinet_pcb/connectors.kicad_sch (KiCad schematic)
At the start: 9 parts, among them J10 Conn_02x05_Odd_Even, J6 Conn_02x09_Odd_Even, J7 Screw_Terminal_01x02, J8 Conn_01x06_Pin, J9 Conn_01x02_Socket

Commit message: PCB Update for package
Parts:
- removed J9: Conn_01x02_Socket, Connector_PinHeader_2.54mm:PinHeader_1x02_P2.54mm_Vertical, symbol Connector:Conn_01x02_Socket
Changed lines of the file:
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@@
-	(wire
-		(pts
-			(xy 35.56 77.47) (xy 43.18 77.47)
-		)
-		(stroke
-			(width 0)
-			(type default)
-		)
-	)
 	(wire
 		(pts
@@
 		(pts
 			(xy 149.86 121.92) (xy 149.86 124.46)
-		)
-		(stroke
-			(width 0)
-			(type default)
-		)
-	)
-	(wire
-		(pts
-			(xy 35.56 80.01) (xy 43.18 80.01)
 		)
 		(stroke
@@
 	(rectangle
 		(start 16.51 49.53)
-		(end 82.55 90.17)
+		(end 82.55 78.74)
 		(stroke
 			(width 0.635)
@@
 		)
 	)
-	(hierarchical_label "LOCK_N"
-		(shape input)
-		(at 35.56 80.01 180)
+	(hierarchical_label "GPIO_1"
+		(shape input)
+		(at 129.54 109.22 180)
 		(fields_autoplaced yes)
 		(effects
@@
 		)
 	)
-	(hierarchical_label "GPIO_1"
-		(shape input)
-		(at 129.54 109.22 180)
+	(hierarchical_label "GPIO_3"
+		(shape input)
+		(at 129.54 114.3 180)
 		(fields_autoplaced yes)
 		(effects
@@
 		)
 	)
-	(hierarchical_label "GPIO_3"
-		(shape input)
-		(at 129.54 114.3 180)
-		(fields_autoplaced yes)
-		(effects
-			(font
-				(size 1.27 1.27)
-			)
-			(justify right)
-		)
-	)
 	(hierarchical_label "JTAG_MTMS"
 		(shape input)
@@
 			)
 			(justify left)
-		)
-	)
-	(hierarchical_label "LOCK_P"
-		(shape input)
-		(at 35.56 77.47 180)
-		(fields_autoplaced yes)
-		(effects
-			(font
-				(size 1.27 1.27)
-			)
-			(justify right)
 		)
 	)
@@
 					(unit 1)
 				)
-			)
-		)
-	)
-	(symbol
-		(lib_id "Connector:Conn_01x02_Socket")
-		(at 48.26 77.47 0)
-		(unit 1)
-		(exclude_from_sim no)
-		(in_bom yes)
-		(on_board yes)
-		(dnp no)
-		(fields_autoplaced yes)
-		(property "Reference" "J9"
-			(at 49.53 77.4699 0)
-			(effects
-				(font
-					(size 1.27 1.27)
-				)
-				(justify left)
-			)
-		)
-		(property "Value" "Conn_01x02_Socket"
-			(at 49.53 80.0099 0)
-			(effects
-				(font
-					(size 1.27 1.27)
-				)
-				(justify left)
-			)
-		)
-		(property "Footprint" "Connector_PinHeader_2.54mm:PinHeader_1x02_P2.54mm_Vertical"
-			(at 48.26 77.47 0)
-			(effects
-				(font
-					(size 1.27 1.27)
-				)
-				(hide yes)
-			)
-		)
-		(property "Datasheet" "~"
-			(at 48.26 77.47 0)
-			(effects
-				(font
-					(size 1.27 1.27)
-				)
-				(hide yes)
-			)
-		)
-		(property "Description" "Generic connector, single row, 01x02, script generated"
-			(at 48.26 77.47 0)
-			(effects
-				(font
-					(size 1.27 1.27)
-				)
-				(hide yes)
-			)
-		)
-		(pin "2"
-		)
-		(pin "1"
-		)
-		(instances
-			(project "onyks_iot_control_cabinet_pcb"
-				(path "/789878cb-67d5-4bc7-a42d-b3bc72d661d0/9fa608f4-5282-4caa-ae1b-46582b97cb5d"
-					(reference "J9")
-					(unit 1)
-				)
