File: pcb/onyks_iot_control_cabinet_pcb/Power_Supply.kicad_sch (KiCad schematic)
At the start: 23 parts, among them IC1 TPS54231DR, J3 Screw_Terminal_01x02, J4 Jack-DC, J5 Conn_01x03_Pin, U2 LM1117MP-3.3

Commit message: PCB Ressurection
Parts:
- removed J4: Jack-DC, Connector_BarrelJack:BarrelJack_CLIFF_FC681465S_SMT_Horizontal, symbol Connector:Jack-DC
- added J4: Barrel_Jack_Switch, Connector_BarrelJack:BarrelJack_CLIFF_FC681465S_SMT_Horizontal, symbol Connector:Barrel_Jack_Switch
- J5: footprint Connector_PinHeader_2.54mm:PinHeader_1x03_P2.54mm_Horizontal -> Connector_PinHeader_2.54mm:PinHeader_1x03_P2.54mm_Vertical
- L1: value L -> 15u
- renumbered C9 to C10, C10 to C11, C14 to C12, C11 to C13, C13 to C14, C12 to C8, C8 to C9
Connections:
- net GND: now also J4.2, J4.3
- net at J5.1 (Pin_1): now also J4.1
Other:
- moved on the sheet: C10, C11, C12, C13, C14, C15, C5, C6, C7, C8, C9, D2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
