File: pcb/onyks_iot_control_cabinet_pcb/MCU.kicad_sch (KiCad schematic)
At the start: 14 parts, among them J1 Conn_02x05_Odd_Even, J2 Conn_01x06_Pin, Q1 BC847B, Q2 BC847B, SW1 SW_Push, SW2 SW_Push, U1 ESP32-WROOM-32D

Commit message: PCB Update
Connections:
- removed net GPIO_1: U1.24 (IO2), U1.26 (IO4), U1.27 (IO16)
- net GPIO_3 renamed GPIO_O3
- net GPIO_O3: no longer U1.9 (IO33)
- net GPIO_6 renamed GPIO_O6
- net GPIO_7 renamed GPIO_O7
- new net GPIO_O1: U1.24 (IO2)
- new net GPIO_O2: U1.26 (IO4)
- new net GPIO_O4: U1.27 (IO16)
- new net GPIO_O5: U1.9 (IO33)
Changed lines of the file:
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@@
+	(wire
+		(pts
+			(xy 138.43 90.17) (xy 151.13 90.17)
+		)
+		(stroke
+			(width 0)
+			(type default)
+		)
+	)
 	(wire
 		(pts
@@
 		(pts
 			(xy 134.62 59.69) (xy 138.43 59.69)
-		)
-		(stroke
-			(width 0)
-			(type default)
-		)
-	)
-	(wire
-		(pts
-			(xy 138.43 90.17) (xy 151.13 90.17)
 		)
 		(stroke
@@
 		)
 	)
+	(label "MTMS"
+		(at 62.23 40.64 180)
+		(effects
+			(font
+				(size 1.27 1.27)
+			)
+			(justify right bottom)
+		)
+	)
+	(label "MTDI"
+		(at 62.23 35.56 180)
+		(effects
+			(font
+				(size 1.27 1.27)
+			)
+			(justify right bottom)
+		)
+	)
+	(label "MCU_RESET"
+		(at 76.2 186.69 180)
+		(effects
+			(font
+				(size 1.27 1.27)
+			)
+			(justify right bottom)
+		)
+	)
+	(label "MTMS"
+		(at 149.86 97.79 180)
+		(effects
+			(font
+				(size 1.27 1.27)
+			)
+			(justify right bottom)
+		)
+	)
+	(label "MCU_RESET"
+		(at 71.12 105.41 180)
+		(effects
+			(font
+				(size 1.27 1.27)
+			)
+			(justify right bottom)
+		)
+	)
+	(label "MTDO"
+		(at 62.23 43.18 180)
+		(effects
+			(font
+				(size 1.27 1.27)
+			)
+			(justify right bottom)
+		)
+	)
 	(label "GPIO_5"
 		(at 149.86 90.17 180)
@@
 		)
 	)
+	(label "GPIO_27"
+		(at 149.86 125.73 180)
+		(effects
+			(font
+				(size 1.27 1.27)
+			)
+			(justify right bottom)
+		)
+	)
+	(label "RTS"
+		(at 44.45 82.55 0)
+		(effects
+			(font
+				(size 1.27 1.27)
+			)
+			(justify left bottom)
+		)
+	)
+	(label "RXD"
+		(at 149.86 85.09 180)
+		(effects
+			(font
+				(size 1.27 1.27)
+			)
+			(justify right bottom)
+		)
+	)
+	(label "GPIO_18"
+		(at 149.86 107.95 180)
+		(effects
+			(font
+				(size 1.27 1.27)
+			)
+			(justify right bottom)
+		)
+	)
+	(label "GPIO_26"
+		(at 149.86 123.19 180)
+		(effects
+			(font
+				(size 1.27 1.27)
+			)
+			(justify right bottom)
+		)
+	)
+	(label "MTDI"
+		(at 149.86 92.71 180)
+		(effects
+			(font
+				(size 1.27 1.27)
+			)
+			(justify right bottom)
+		)
+	)
+	(label "DTR"
+		(at 44.45 80.01 0)
+		(effects
+			(font
+				(size 1.27 1.27)
+			)
+			(justify left bottom)
+		)
+	)
+	(label "DTR"
+		(at 31.75 177.8 0)
+		(effects
+			(font
+				(size 1.27 1.27)
+			)
+			(justify left bottom)
+		)
+	)
 	(label "GPIO_4"
 		(at 149.86 87.63 180)
@@
 		)
 	)
-	(label "MTMS"
-		(at 62.23 40.64 180)
-		(effects
-			(font
-				(size 1.27 1.27)
-			)
-			(justify right bottom)
-		)
-	)
-	(label "MTDI"
-		(at 62.23 35.56 180)
-		(effects
-			(font
-				(size 1.27 1.27)
-			)
-			(justify right bottom)
-		)
-	)
-	(label "MCU_RESET"
-		(at 76.2 186.69 180)
-		(effects
-			(font
-				(size 1.27 1.27)
-			)
-			(justify right bottom)
-		)
-	)
-	(label "MTMS"
-		(at 149.86 97.79 180)
-		(effects
-			(font
-				(size 1.27 1.27)
-			)
-			(justify right bottom)
-		)
-	)
-	(label "MCU_RESET"
-		(at 71.12 105.41 180)
-		(effects
-			(font
-				(size 1.27 1.27)
-			)
-			(justify right bottom)
-		)
-	)
-	(label "MTDO"
-		(at 62.23 43.18 180)
-		(effects
-			(font
-				(size 1.27 1.27)
-			)
-			(justify right bottom)
-		)
-	)
-	(label "GPIO_27"
-		(at 149.86 125.73 180)
-		(effects
-			(font
-				(size 1.27 1.27)
-			)
-			(justify right bottom)
-		)
-	)
-	(label "RTS"
-		(at 44.45 82.55 0)
-		(effects
-			(font
-				(size 1.27 1.27)
-			)
-			(justify left bottom)
-		)
-	)
-	(label "RXD"
-		(at 149.86 85.09 180)
-		(effects
-			(font
-				(size 1.27 1.27)
-			)
-			(justify right bottom)
-		)
-	)
-	(label "GPIO_18"
-		(at 149.86 107.95 180)
-		(effects
-			(font
-				(size 1.27 1.27)
-			)
-			(justify right bottom)
-		)
-	)
-	(label "GPIO_26"
-		(at 149.86 123.19 180)
-		(effects
-			(font
-				(size 1.27 1.27)
-			)
-			(justify right bottom)
-		)
-	)
-	(label "MTDI"
-		(at 149.86 92.71 180)
-		(effects
-			(font
-				(size 1.27 1.27)
-			)
-			(justify right bottom)
-		)
-	)
-	(label "DTR"
-		(at 44.45 80.01 0)
-		(effects
-			(font
-				(size 1.27 1.27)
-			)
-			(justify left bottom)
-		)
-	)
-	(label "DTR"
-		(at 31.75 177.8 0)
-		(effects
-			(font
-				(size 1.27 1.27)
-			)
-			(justify left bottom)
-		)
-	)
 	(label "RTS"
 		(at 31.75 157.48 0)
@@
 		)
 	)
-	(hierarchical_label "GPIO_4"
+	(hierarchical_label "GPIO_O4"
 		(shape input)
 		(at 151.13 102.87 0)
@@
 		)
 	)
-	(hierarchical_label "GPIO_6"
+	(hierarchical_label "GPIO_O6"
 		(shape input)
 		(at 151.13 133.35 0)
@@
 		)
 	)
-	(hierarchical_label "GPIO_2"
+	(hierarchical_label "GPIO_O2"
 		(shape input)
 		(at 151.13 87.63 0)
@@
 		)
 	)
-	(hierarchical_label "GPIO_5"
+	(hierarchical_label "GPIO_O3"
+		(shape input)
+		(at 151.13 90.17 0)
+		(effects
+			(font
+				(size 1.27 1.27)
+			)
+			(justify left)
+		)
+	)
+	(hierarchical_label "GPIO_O5"
 		(shape input)
 		(at 151.13 130.81 0)
@@
 		)
 	)
-	(hierarchical_label "GPIO_3"
-		(shape input)
-		(at 151.13 90.17 0)
-		(effects
-			(font
-				(size 1.27 1.27)
-			)
-			(justify left)
-		)
-	)
 	(hierarchical_label "LOCK_SWITCH"
 		(shape input)
@@
 		)
 	)
-	(hierarchical_label "GPIO_1"
+	(hierarchical_label "GPIO_O1"
 		(shape input)
 		(at 151.13 82.55 0)
@@
 		)
 	)
-	(hierarchical_label "GPIO_7"
+	(hierarchical_label "GPIO_O7"
 		(shape input)
 		(at 151.13 135.89 0)
